Commit message: better URDF definition minor change in make file

File: src/lsbot/lsbot_description/urdf/lidar.urdf.xacro (robot description, xacro)
@@ -73,8 +73,8 @@
           <ros>
             <namespace>/</namespace>
-            <frame_name>${name}</frame_name>
             <remapping>~/out:=${topic}</remapping>
           </ros>
           <output_type>sensor_msgs/LaserScan</output_type>
+          <frame_name>${name}</frame_name>
         </plugin>
       </sensor>

File: src/lsbot/lsbot_description/urdf/sandbox_bot.xacro (robot description, xacro)
@@ -23,5 +23,5 @@
   <xacro:property name="tower_x"        value="${body_length/2 + 0.05}" />
   <xacro:property name="tower_xyz"      value="${tower_x} 0 ${tower_length/2}" />
-  <xacro:property name="tower_mass"     value="0.3" />
+  <xacro:property name="tower_mass"     value="0.05" />
   <!-- Wheel properties
        hub_dia and tire_dia are the diameters of the hub and tire,
@@ -41,5 +41,5 @@
   <!-- Sensor position properties -->
   <xacro:property name="scanner_length"  value="0.07570"/>
-  <xacro:property name="scanner_mass"    value="0.2"/>
+  <xacro:property name="scanner_mass"    value="0.05"/>
   <xacro:property name="sensor_colour"   value="0.8 0 0 1"/>
   <xacro:property name="scanner_width"   value="0.07570"/>
@@ -250,6 +250,5 @@
     <!-- Differential Drive -->
     <plugin name="differential_drive_controller" filename="libgazebo_ros_diff_drive.so">
-      <alwaysOn>true</alwaysOn>
-      <updateRate>40</updateRate>
+      <update_rate>10</update_rate>
       <legacyMode>false</legacyMode>
       <left_joint>left_bogie_rear_axle</left_joint>
@@ -257,22 +256,18 @@
       <wheel_separation>0.4</wheel_separation>
       <wheel_diameter>0.2</wheel_diameter>
-      <max_wheel_torque>10</max_wheel_torque>
+      <max_wheel_torque>100</max_wheel_torque>
       <max_wheel_acceleration>1.0</max_wheel_acceleration>
-      <commandTopic>cmd_vel</commandTopic>
-      <odometryTopic>odom</odometryTopic>
-      <odometryFrame>odom</odometryFrame>
-      <robotBaseFrame>robot_footprint</robotBaseFrame>
-      <publishWheelTF>true</publishWheelTF>
-      <publishWheelJointState>false</publishWheelJointState>
-      <rosDebugLevel>na</rosDebugLevel>
-      <wheelAcceleration>0</wheelAcceleration>
-      <wheelTorque>5</wheelTorque>
-      <odometrySource>world</odometrySource>
+      <command_topic>cmd_vel</command_topic>
       <publish_odom>true</publish_odom>
-      <publish_odom_tf>true</publish_odom_tf>
-      <robotNamespace>/</robotNamespace>
-      <broadcastTF>1</broadcastTF>
+      <publish_odom_tf>false</publish_odom_tf>
+      <publish_wheel_tf>true</publish_wheel_tf>
+      <odometry_topic>odom</odometry_topic>
       <odometry_frame>odom</odometry_frame>
       <robot_base_frame>robot_footprint</robot_base_frame>
+      <odometry_source>1</odometry_source>
+      <ros>
+        <namespace>/</namespace>
+        <remapping>odom:=odom_shaft</remapping>
+      </ros>
     </plugin>
   </gazebo>

Commit message: migration to ROS melodic

File: src/lsbot/lsbot_description/urdf/lidar.urdf.xacro (robot description, xacro)
@@ -34,5 +34,5 @@
     </link>
   </xacro:macro>
-  <xacro:macro name="lidar" params="name parent width height position samples angle topic orientation">
+  <xacro:macro name="lidar" params="name parent width height position samples angle topic orientation frame">
     <link name="${name}">
       <visual>
@@ -70,11 +70,7 @@
           </range>
         </ray>
-        <plugin name="gazebo_ros_${name}_hokuyo_controller" filename="libgazebo_ros_ray_sensor.so">
-          <ros>
-            <namespace>/</namespace>
-            <remapping>~/out:=${topic}</remapping>
-          </ros>
-          <output_type>sensor_msgs/LaserScan</output_type>
-          <frame_name>${name}</frame_name>
+        <plugin name="gazebo_ros_${name}_hokuyo_controller" filename="libgazebo_ros_laser.so">
+          <topicName>${topic}</topicName>
+          <frameName>${frame}</frameName>
         </plugin>
       </sensor>

File: src/lsbot/lsbot_description/urdf/lsbot.xacro (robot description, xacro)
@@ -321,6 +321,6 @@
         <argument>--ros-args --remap ~/out:=${prefix}joint_states</argument>
       </ros>
-      <update_rate>10</update_rate>
-      <joint_name>${prefix}motor1</joint_name>
+      <updateRate>10</updateRate>
+      <jointName>${prefix}motor1</jointName>
     </plugin>
     <plugin name="lsbot_actuator_rotaryservo" filename="liblsbot_gazebo_joint_plugin.so">
@@ -330,24 +330,26 @@
     <!-- Differential Drive -->
     <plugin name="differential_drive_controller" filename="libgazebo_ros_diff_drive.so">
-      <update_rate>10</update_rate>
+      <rosDebugLevel>na</rosDebugLevel>
       <legacyMode>false</legacyMode>
-      <left_joint>left_bogie_rear_axle</left_joint>
-      <right_joint>right_bogie_rear_axle</right_joint>
-      <wheel_separation>0.4</wheel_separation>
-      <wheel_diameter>0.2</wheel_diameter>
-      <max_wheel_torque>100</max_wheel_torque>
-      <max_wheel_acceleration>1.0</max_wheel_acceleration>
-      <command_topic>cmd_vel</command_topic>
-      <publish_odom>true</publish_odom>
-      <publish_odom_tf>false</publish_odom_tf>
-      <publish_wheel_tf>true</publish_wheel_tf>
-      <odometry_topic>odom</odometry_topic>
-      <odometry_frame>odom</odometry_frame>
-      <robot_base_frame>robot_footprint</robot_base_frame>
-      <odometry_source>1</odometry_source>
-      <ros>
-        <namespace>/</namespace>
-        <remapping>odom:=odom_shaft</remapping>
-      </ros>
+      <publishWheelTF>true</publishWheelTF>
+      <robotNamespace>/</robotNamespace>
+      <publishTf>1</publishTf>
+      <publishOdomTF>0</publishOdomTF>
+      <publishWheelJointState>true</publishWheelJointState>
+      <alwaysOn>true</alwaysOn>
+      <updateRate>5</updateRate>
+      <leftJoint>left_bogie_rear_axle</leftJoint>
+      <rightJoint>right_bogie_rear_axle</rightJoint>
+      <wheelSeparation>0.4</wheelSeparation>
+      <wheelDiameter>0.2</wheelDiameter>
+      <broadcastTF>1</broadcastTF>
+      <wheelTorque>2800</wheelTorque>
+      <wheelAcceleration>1.0</wheelAcceleration>
+      <commandTopic>cmd_vel</commandTopic>
+      <odometryFrame>odom</odometryFrame>
+      <odometryTopic>odom_shaft</odometryTopic>
+      <robotBaseFrame>robot_footprint</robotBaseFrame>
+      <odometrySource>world</odometrySource>
+      <!--odometrysource>1</odometry_source-->
     </plugin>
   </gazebo>
@@ -357,5 +359,5 @@
     <origin xyz="${scanner_position}" rpy="0 0 0"/>
   </xacro:lidar-->
-  <xacro:lidar name="scanner" parent="body" width="${scanner_width}" height="${scanner_height}" position="${scanner_position}" samples="${scanner_samples}" angle="${scanner_angle}" topic="${scanner_topic}" orientation="${scanner_orientation}" />
-  <xacro:lidar name="floorscan" parent="motor1_cover" width="${scanner_width}" height="${scanner_height}" position="${floorscanner_position_rotate}" samples="${scanner_samples}" angle="${floorscanner_angle}" topic="${floorscanner_topic}" orientation="${floorscanner_orientation_rotate}" />
+  <xacro:lidar name="scanner" parent="body" width="${scanner_width}" height="${scanner_height}" position="${scanner_position}" samples="${scanner_samples}" angle="${scanner_angle}" topic="${scanner_topic}" orientation="${scanner_orientation}" frame="scanner"/>
+  <xacro:lidar name="floorscan" parent="motor1_cover" width="${scanner_width}" height="${scanner_height}" position="${floorscanner_position_rotate}" samples="${scanner_samples}" angle="${floorscanner_angle}" topic="${floorscanner_topic}" orientation="${floorscanner_orientation_rotate}" frame="floorscan_dynamic"/>
 </robot>
